File: Hardware/Project_KiCad6/CO2Guard/CO2Guard.kicad_pcb (KiCad board)
At the start: 2 copper layers, 62.3 x 64.2 mm, 24 parts, among them K1 Conn_01x03, K2 Conn_01x04, T1 BC327

Commit message: Added Enclosure
Other:
- board text added: "V 2.1 KiCad Edition 210043-1"
- board text removed: "V 2.1 KiCad Edition"
Changed lines of the file:
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@@
   (paper "A4")
   (title_block
-    (comment 4 "AISLER Project ID: GOOGJQGG")
+    (title "Elektor CO2 Meter (210043)")
+    (date "2022-01-14")
+    (company "Elektor Labs")
+    (comment 4 "AISLER Project ID: ZKYMXGLS")
   )
   (layers
@@
     (property "Sheetfile" "CO2Guard.kicad_sch")
     (property "Sheetname" "")
+    (property "mpn" "LR0204F1K5")
     (attr through_hole)
     (fp_text reference "R1" (at 0.3556 1.5748) (layer "F.SilkS")
@@
     (property "Sheetfile" "CO2Guard.kicad_sch")
     (property "Sheetname" "")
+    (property "mpn" "151031SS04000")
     (attr through_hole)
     (fp_text reference "D2" (at -0.9652 -0.0508 180) (layer "F.SilkS")
@@
     (property "Sheetfile" "CO2Guard.kicad_sch")
     (property "Sheetname" "")
+    (property "mpn" "WT-1205")
     (attr through_hole)
     (fp_text reference "BZ1" (at 3.8 -7.2 180) (layer "F.SilkS")
@@
     (property "Sheetfile" "CO2Guard.kicad_sch")
     (property "Sheetname" "")
+    (property "mpn" "MBA02040C3300FRP00")
     (attr through_hole)
     (fp_text reference "R5" (at -1.6764 -0.3048 180) (layer "F.SilkS")
@@
     (property "Sheetfile" "CO2Guard.kicad_sch")
     (property "Sheetname" "")
+    (property "mpn" "MKS2C031001A00KSSD")
     (attr through_hole)
     (fp_text reference "C3" (at -2.3876 0) (layer "F.SilkS")
@@
     (fp_arc (start -1.37 -6.21) (mid -0.784214 -7.624214) (end 0.63 -8.21) (layer "F.Fab") (width 0.1))
     (pad "1" thru_hole rect locked (at 0 0) (size 2 2) (drill 1) (layers *.Cu *.Mask)
-      (net 21 "unconnected-(MOD2-Pad1)") (pinfunction "~RST") (pintype "input"))
+      (net 21 "unconnected-(MOD2-Pad1)") (pinfunction "~{RST}") (pintype "input"))
     (pad "2" thru_hole oval locked (at 0 2.54) (size 2 1.6) (drill 1) (layers *.Cu *.Mask)
       (net 25 "unconnected-(MOD2-Pad2)") (pinfunction "A0") (pintype "input"))
@@
     (property "Sheetfile" "CO2Guard.kicad_sch")
     (property "Sheetname" "")
+    (property "mpn" "151031YS06000")
     (attr through_hole)
     (fp_text reference "D3" (at -1.0668 -0.1524) (layer "F.SilkS")
@@
     (property "Sheetfile" "CO2Guard.kicad_sch")
     (property "Sheetname" "")
+    (property "mpn" "BAT85S-TR")
     (attr through_hole)
     (fp_text reference "D1" (at 0.0508 1.27) (layer "F.SilkS")
@@
     (property "Sheetfile" "CO2Guard.kicad_sch")
     (property "Sheetname" "")
+    (property "mpn" "BC32725BU")
     (attr through_hole)
     (fp_text reference "T1" (at -2.53754 0.03993) (layer "F.SilkS")
@@
     (property "Sheetfile" "CO2Guard.kicad_sch")
     (property "Sheetname" "")
+    (property "mpn" "860020573008")
     (attr through_hole)
     (fp_text reference "C1" (at 3.8608 -3.556 -90) (layer "F.SilkS")
@@
     (property "Sheetfile" "CO2Guard.kicad_sch")
     (property "Sheetname" "")
+    (property "mpn" "ZR0207C")
     (attr through_hole)
     (fp_text reference "R3" (at 7.5184 3.3528) (layer "F.SilkS")
@@
     (property "Sheetfile" "CO2Guard.kicad_sch")
     (property "Sheetname" "")
+    (property "mpn" "CFR-25JB-52-4K7")
     (attr through_hole)
     (fp_text reference "R2" (at 8.4836 2.2352) (layer "F.SilkS")
@@
     (property "Sheetfile" "CO2Guard.kicad_sch")
     (property "Sheetname" "")
+    (property "mpn" "MBA02040C3300FRP00")
     (attr through_hole)
     (fp_text reference "R4" (at -1.6764 0) (layer "F.SilkS")
@@
     (property "Sheetfile" "CO2Guard.kicad_sch")
     (property "Sheetname" "")
+    (property "mpn" "ZR0207C")
     (attr through_hole)
     (fp_text reference "R7" (at 0.3556 1.4224) (layer "F.SilkS")
@@
     (property "Sheetfile" "CO2Guard.kicad_sch")
     (property "Sheetname" "")
+    (property "mpn" "MBA02040C3300FRP00")
     (attr through_hole)
     (fp_text reference "R6" (at -1.6764 -0.254 180) (layer "F.SilkS")
@@
     (property "Sheetfile" "CO2Guard.kicad_sch")
     (property "Sheetname" "")
+    (property "mpn" "MKS2C031001A00KSSD")
     (attr through_hole)
     (fp_text reference "C2" (at -2.5184 -0.7112) (layer "F.SilkS")
@@
     (property "Sheetfile" "CO2Guard.kicad_sch")
     (property "Sheetname" "")
+    (property "mpn" "151031VS06000")
     (attr through_hole)
     (fp_text reference "D4" (at -0.8636 0) (layer "F.SilkS")
@@
   (gr_line (start 155.8544 137.1092) (end 155.8036 72.9488) (layer "Edge.Cuts") (width 0.1))
   (gr_line (start 155.8036 72.9488) (end 93.5736 72.9488) (layer "Edge.Cuts") (width 0.1))
-  (gr_text "V 2.1\nKiCad Edition" (at 122.2756 117.0432) (layer "F.Cu")
+  (gr_text "V 2.1\nKiCad Edition\n210043-1\n" (at 122.174 118.364) (layer "F.Cu")
     (effects (font (size 1.5 1.5) (thickness 0.3)))
   )
@@
     (polygon
       (pts
-        (xy 130.1496 119.5832)
-        (xy 114.1984 119.5832)
-        (xy 114.2492 113.7412)
-        (xy 130.2004 113.7412)
+        (xy 130.1242 124.587)
+        (xy 114.173 124.587)
+        (xy 114.2238 113.665)
+        (xy 130.175 113.665)
       )
     )
