File: Hardware/Project_KiCad6/CO2Guard/CO2Guard.kicad_sch (KiCad schematic)
At the start: 24 parts, among them K1 Conn_01x03, K2 Conn_01x04, T1 BC327

Commit message: added MPN to schematic parts
Parts:
- BZ1: mpn (none) -> WT-1205
- C1: mpn (none) -> 860020573008
- C2, C3: mpn (none) -> MKS2C031001A00KSSD
- D1: mpn (none) -> BAT85S-TR
- D2: mpn (none) -> 151031SS04000
- D3: mpn (none) -> 151031YS06000
- D4: mpn (none) -> 151031VS06000
- R1: mpn (none) -> LR0204F1K5
- R2: mpn (none) -> CFR-25JB-52-4K7
- R3, R7: mpn (none) -> ZR0207C
- R4, R5, R6: mpn (none) -> MBA02040C3300FRP00
- T1: mpn (none) -> BC32725BU
Changed lines of the file:
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@@
+      (effects (font (size 1.27 1.27)) hide)
+    )
+    (property "mpn" "MBA02040C3300FRP00" (id 4) (at 113.03 39.37 90)
       (effects (font (size 1.27 1.27)) hide)
     )
@@
     )
     (property "Datasheet" "~" (id 3) (at 63.5 33.02 0)
+      (effects (font (size 1.27 1.27)) hide)
+    )
+    (property "mpn" "860020573008" (id 4) (at 63.5 33.02 0)
       (effects (font (size 1.27 1.27)) hide)
     )
@@
       (effects (font (size 1.27 1.27)) hide)
     )
+    (property "mpn" "151031YS06000" (id 4) (at 101.6 30.48 0)
+      (effects (font (size 1.27 1.27)) hide)
+    )
     (pin "1")
     (pin "2")
@@
     )
     (property "Datasheet" "~" (id 3) (at 67.31 74.93 0)
+      (effects (font (size 1.27 1.27)) hide)
+    )
+    (property "mpn" "CFR-25JB-52-4K7" (id 4) (at 67.31 74.93 0)
       (effects (font (size 1.27 1.27)) hide)
     )
@@
       (effects (font (size 1.27 1.27)) hide)
     )
+    (property "mpn" "WT-1205" (id 4) (at 50.8 80.01 0)
+      (effects (font (size 1.27 1.27)) hide)
+    )
     (pin "1")
     (pin "2")
@@
     )
     (property "Datasheet" "~" (id 3) (at 113.03 30.48 0)
+      (effects (font (size 1.27 1.27)) hide)
+    )
+    (property "mpn" "MBA02040C3300FRP00" (id 4) (at 113.03 30.48 90)
       (effects (font (size 1.27 1.27)) hide)
     )
@@
       (effects (font (size 1.27 1.27)) hide)
     )
+    (property "mpn" "MKS2C031001A00KSSD" (id 4) (at 63.5 81.28 0)
+      (effects (font (size 1.27 1.27)) hide)
+    )
     (pin "1")
     (pin "2")
@@
     )
     (property "Datasheet" "~" (id 3) (at 67.31 64.77 0)
+      (effects (font (size 1.27 1.27)) hide)
+    )
+    (property "mpn" "LR0204F1K5" (id 4) (at 67.31 64.77 0)
       (effects (font (size 1.27 1.27)) hide)
     )
@@
       (effects (font (size 1.27 1.27)) hide)
     )
+    (property "mpn" "151031SS04000" (id 4) (at 101.6 22.225 0)
+      (effects (font (size 1.27 1.27)) hide)
+    )
     (pin "1")
     (pin "2")
@@
     (property "Datasheet" "http://www.onsemi.com/pub_link/Collateral/BC327-D.PDF" (id 3) (at 55.88 69.85 0)
       (effects (font (size 1.27 1.27)) (justify left) hide)
+    )
+    (property "mpn" "BC32725BU" (id 4) (at 55.88 69.85 0)
+      (effects (font (size 1.27 1.27)) hide)
     )
     (pin "1")
@@
       (effects (font (size 1.27 1.27)) hide)
     )
+    (property "mpn" "ZR0207C" (id 4) (at 69.85 30.48 90)
+      (effects (font (size 1.27 1.27)) hide)
+    )
     (pin "1")
     (pin "2")
@@
       (effects (font (size 1.27 1.27)) hide)
     )
+    (property "mpn" "ZR0207C" (id 4) (at 163.83 71.755 90)
+      (effects (font (size 1.27 1.27)) hide)
+    )
     (pin "1")
     (pin "2")
@@
       (effects (font (size 1.27 1.27)) hide)
     )
+    (property "mpn" "BAT85S-TR" (id 4) (at 55.88 80.01 0)
+      (effects (font (size 1.27 1.27)) hide)
+    )
     (pin "1")
     (pin "2")
@@
       (effects (font (size 1.27 1.27)) hide)
     )
+    (property "mpn" "151031VS06000" (id 4) (at 102.235 39.37 0)
+      (effects (font (size 1.27 1.27)) hide)
+    )
     (pin "1")
     (pin "2")
@@
       (effects (font (size 1.27 1.27)) hide)
     )
+    (property "mpn" "MBA02040C3300FRP00" (id 4) (at 113.03 22.225 90)
+      (effects (font (size 1.27 1.27)) hide)
+    )
     (pin "1")
     (pin "2")
@@
       (effects (font (size 1.27 1.27)) hide)
     )
+    (property "mpn" "MKS2C031001A00KSSD" (id 4) (at 200.66 30.48 0)
+      (effects (font (size 1.27 1.27)) hide)
+    )

Commit message: Added Enclosure
Other:
- company: (none) -> Elektor Labs
- title: (none) -> Elektor CO2 Guard (210043)
Changed lines of the file:
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@@
 (kicad_sch (version 20211123) (generator eeschema)
   (paper "A4")
+  (title_block
+    (title "Elektor CO2 Guard (210043)")
+    (company "Elektor Labs")
+  )
   (junction (at 177.8 19.05) (diameter 1.016) (color 0 0 0 0)
   )
